File: EVSE-Car-Simulator/EVSE-Car-Simulator.kicad_pcb (KiCad board)
At the start: 2 copper layers, 36.8 x 17.8 mm, 10 parts, among them J1 E, J2 A/B, J3 D-fault, J4 C, J5 Type 2, J6 CP Diag

Commit message: open files in kicad8
Other:
- net class Default removed
